Commit message: the ball is being picked!

File: fh_description/smart_grasping_sandbox.urdf (robot description, URDF)
Before this commit: robot ur10, 36 links, 35 joints
Joints:
- joint H1_F1J1: limit lower=-1.57079632679 upper=1.0472 effort=2 velocity=1.0 -> lower=-1.57079632679 upper=1.0472 effort=50 velocity=1.0
- joint H1_F1J2: limit lower=-1.04716 upper=1.57075 effort=2 velocity=1.0 -> lower=-1.04716 upper=1.57075 effort=50 velocity=1.0
- joint H1_F2J1: limit lower=-1.57079632679 upper=1.0472 effort=2 velocity=1.0 -> lower=-1.57079632679 upper=1.0472 effort=30 velocity=1.0
- joint H1_F2J2: limit lower=-1.04716 upper=1.57075 effort=2 velocity=1.0 -> lower=-1.04716 upper=1.57075 effort=30 velocity=1.0
- joint H1_F3J1: limit lower=-1.57079632679 upper=1.0472 effort=2 velocity=1.0 -> lower=-1.57079632679 upper=1.0472 effort=30 velocity=1.0
- joint H1_F3J2: limit lower=-1.04716 upper=1.57075 effort=2 velocity=1.0 -> lower=-1.04716 upper=1.57075 effort=30 velocity=1.0
- joint H1_WRJ1: limit lower=-0.785 upper=0.785 effort=20 velocity=0.1 -> lower=-0.785 upper=0.785 effort=50 velocity=0.1
