Commit message: Adding dat files, modified Dockerfile. Gzweb is still not working

File: fh_desc/smart_grasping_sandbox.urdf (robot description, URDF)
Before this commit: robot ur10, 36 links, 35 joints
Links:
- link H1_F1_base_link: geometry collision mesh filename=model://fh_desc/meshes/base_link.dae; visual mesh filename=model://fh_desc/meshes/base_link.dae
- link H1_F1_link_1: geometry collision mesh filename=model://fh_desc/meshes/prox.dae; visual mesh filename=model://fh_desc/meshes/prox.dae
- link H1_F1_link_2: geometry collision mesh filename=model://fh_desc/meshes/dist.dae; visual mesh filename=model://fh_desc/meshes/dist.dae
- link H1_F1_tip: geometry collision mesh filename=model://fh_desc/meshes/omd-d18-tip.dae; visual mesh filename=model://fh_desc/meshes/omd-d18-tip.dae
- link H1_F2_base_link: geometry collision mesh filename=model://fh_desc/meshes/base_link.dae; visual mesh filename=model://fh_desc/meshes/base_link.dae
- link H1_F2_link_1: geometry collision mesh filename=model://fh_desc/meshes/prox.dae; visual mesh filename=model://fh_desc/meshes/prox.dae
- link H1_F2_link_2: geometry collision mesh filename=model://fh_desc/meshes/dist.dae; visual mesh filename=model://fh_desc/meshes/dist.dae
- link H1_F2_tip: geometry collision mesh filename=model://fh_desc/meshes/omd-d18-tip.dae; visual mesh filename=model://fh_desc/meshes/omd-d18-tip.dae
- link H1_F3_base_link: geometry collision mesh filename=model://fh_desc/meshes/base_link.dae; visual mesh filename=model://fh_desc/meshes/base_link.dae
- link H1_F3_link_1: geometry collision mesh filename=model://fh_desc/meshes/prox.dae; visual mesh filename=model://fh_desc/meshes/prox.dae
- link H1_F3_link_2: geometry collision mesh filename=model://fh_desc/meshes/dist.dae; visual mesh filename=model://fh_desc/meshes/dist.dae
- link H1_F3_tip: geometry collision mesh filename=model://fh_desc/meshes/omd-d18-tip.dae; visual mesh filename=model://fh_desc/meshes/omd-d18-tip.dae
- link H1_WR_force_torque_sensor: geometry collision mesh filename=model://fh_desc/meshes/force_torque_sensor.dae; visual mesh filename=model://fh_desc/meshes/force_torque_sensor.dae
- link H1_WR_wrist: geometry collision mesh filename=model://fh_desc/meshes/wrist.dae; visual mesh filename=model://fh_desc/meshes/wrist.dae
- link H1_WR_wrist_base: geometry collision mesh filename=model://fh_desc/meshes/wrist_base.dae; visual mesh filename=model://fh_desc/meshes/wrist_base.dae
- link H1_base_link: geometry collision mesh filename=model://fh_desc/meshes/palm_base.dae; visual mesh filename=model://fh_desc/meshes/palm_base.dae
- link base_link: geometry collision mesh filename=model://ur_description/meshes/ur10/collision/base.dae; visual mesh filename=model://ur_description/meshes/ur10/visual/base.dae
- link forearm_link: geometry collision mesh filename=model://ur_description/meshes/ur10/collision/forearm.dae; visual mesh filename=model://ur_description/meshes/ur10/visual/forearm.dae
- link shoulder_link: geometry collision mesh filename=model://ur_description/meshes/ur10/collision/shoulder.dae; visual mesh filename=model://ur_description/meshes/ur10/visual/shoulder.dae
- link upper_arm_link: geometry collision mesh filename=model://ur_description/meshes/ur10/collision/upperarm.dae; visual mesh filename=model://ur_description/meshes/ur10/visual/upperarm.dae
- link wrist_1_link: geometry collision mesh filename=model://ur_description/meshes/ur10/collision/wrist1.dae; visual mesh filename=model://ur_description/meshes/ur10/visual/wrist1.dae
- link wrist_2_link: geometry collision mesh filename=model://ur_description/meshes/ur10/collision/wrist2.dae; visual mesh filename=model://ur_description/meshes/ur10/visual/wrist2.dae
- link wrist_3_link: geometry collision mesh filename=model://ur_description/meshes/ur10/collision/wrist3.dae; visual mesh filename=model://ur_description/meshes/ur10/visual/wrist3.dae
