Commit message: Finally spawning in gzweb

File: fh_desc/model.urdf (robot description, URDF)
Before this commit: robot ur10, 36 links, 35 joints
Links:
- link H1_F1_base_link: geometry collision mesh filename=package://fh_desc/meshes/base_link.dae; visual mesh filename=package://fh_desc/meshes/base_link.dae
- link H1_F1_link_1: geometry collision mesh filename=package://fh_desc/meshes/prox.dae; visual mesh filename=package://fh_desc/meshes/prox.dae
- link H1_F1_link_2: geometry collision mesh filename=package://fh_desc/meshes/dist.dae; visual mesh filename=package://fh_desc/meshes/dist.dae
- link H1_F1_tip: geometry collision mesh filename=package://fh_desc/meshes/omd-d18-tip.dae; visual mesh filename=package://fh_desc/meshes/omd-d18-tip.dae
- link H1_F2_base_link: geometry collision mesh filename=package://fh_desc/meshes/base_link.dae; visual mesh filename=package://fh_desc/meshes/base_link.dae
- link H1_F2_link_1: geometry collision mesh filename=package://fh_desc/meshes/prox.dae; visual mesh filename=package://fh_desc/meshes/prox.dae
- link H1_F2_link_2: geometry collision mesh filename=package://fh_desc/meshes/dist.dae; visual mesh filename=package://fh_desc/meshes/dist.dae
- link H1_F2_tip: geometry collision mesh filename=package://fh_desc/meshes/omd-d18-tip.dae; visual mesh filename=package://fh_desc/meshes/omd-d18-tip.dae
- link H1_F3_base_link: geometry collision mesh filename=package://fh_desc/meshes/base_link.dae; visual mesh filename=package://fh_desc/meshes/base_link.dae
- link H1_F3_link_1: geometry collision mesh filename=package://fh_desc/meshes/prox.dae; visual mesh filename=package://fh_desc/meshes/prox.dae
- link H1_F3_link_2: geometry collision mesh filename=package://fh_desc/meshes/dist.dae; visual mesh filename=package://fh_desc/meshes/dist.dae
- link H1_F3_tip: geometry collision mesh filename=package://fh_desc/meshes/omd-d18-tip.dae; visual mesh filename=package://fh_desc/meshes/omd-d18-tip.dae
- link H1_WR_force_torque_sensor: geometry collision mesh filename=package://fh_desc/meshes/force_torque_sensor.dae; visual mesh filename=package://fh_desc/meshes/force_torque_sensor.dae
- link H1_WR_wrist: geometry collision mesh filename=package://fh_desc/meshes/wrist.dae; visual mesh filename=package://fh_desc/meshes/wrist.dae
- link H1_WR_wrist_base: geometry collision mesh filename=package://fh_desc/meshes/wrist_base.dae; visual mesh filename=package://fh_desc/meshes/wrist_base.dae
- link H1_base_link: geometry collision mesh filename=package://fh_desc/meshes/palm_base.dae; visual mesh filename=package://fh_desc/meshes/palm_base.dae
- link base_link: geometry collision mesh filename=package://ur_description/meshes/ur10/collision/base.stl; visual mesh filename=package://ur_description/meshes/ur10/visual/base.dae
- link forearm_link: geometry collision mesh filename=package://ur_description/meshes/ur10/collision/forearm.stl; visual mesh filename=package://ur_description/meshes/ur10/visual/forearm.dae
- link shoulder_link: geometry collision mesh filename=package://ur_description/meshes/ur10/collision/shoulder.stl; visual mesh filename=package://ur_description/meshes/ur10/visual/shoulder.dae
- link upper_arm_link: geometry collision mesh filename=package://ur_description/meshes/ur10/collision/upperarm.stl; visual mesh filename=package://ur_description/meshes/ur10/visual/upperarm.dae
- link wrist_1_link: geometry collision mesh filename=package://ur_description/meshes/ur10/collision/wrist1.stl; visual mesh filename=package://ur_description/meshes/ur10/visual/wrist1.dae
- link wrist_2_link: geometry collision mesh filename=package://ur_description/meshes/ur10/collision/wrist2.stl; visual mesh filename=package://ur_description/meshes/ur10/visual/wrist2.dae
- link wrist_3_link: geometry collision mesh filename=package://ur_description/meshes/ur10/collision/wrist3.stl; visual mesh filename=package://ur_description/meshes/ur10/visual/wrist3.dae
Joints:
- joint world_joint: origin xyz=0.0 0.0 0.0 rpy=0.0 0.0 0.0 -> xyz=0.0 -1.0 1.0 rpy=0.0 0.0 0.0

Commit message: ur10 loads in openrave

File: fh_desc/model.urdf (robot description, URDF)
Before this commit: robot smart_grasping_sandbox, 36 links, 35 joints
Links:
- link base_link: geometry collision mesh filename=package://ur_description/meshes/ur10/collision/base.stl; visual mesh filename=package://ur_description/meshes/ur10/collision/base.stl
- link forearm_link: geometry collision mesh filename=package://ur_description/meshes/ur10/collision/forearm.stl; visual mesh filename=package://ur_description/meshes/ur10/collision/forearm.stl
- link shoulder_link: geometry collision mesh filename=package://ur_description/meshes/ur10/collision/shoulder.stl; visual mesh filename=package://ur_description/meshes/ur10/collision/shoulder.stl
- link upper_arm_link: geometry collision mesh filename=package://ur_description/meshes/ur10/collision/upperarm.stl; visual mesh filename=package://ur_description/meshes/ur10/collision/upperarm.stl
- link wrist_1_link: geometry collision mesh filename=package://ur_description/meshes/ur10/collision/wrist1.stl; visual mesh filename=package://ur_description/meshes/ur10/collision/wrist1.stl
- link wrist_2_link: geometry collision mesh filename=package://ur_description/meshes/ur10/collision/wrist2.stl; visual mesh filename=package://ur_description/meshes/ur10/collision/wrist2.stl
- link wrist_3_link: geometry collision mesh filename=package://ur_description/meshes/ur10/collision/wrist3.stl; visual mesh filename=package://ur_description/meshes/ur10/collision/wrist3.stl

Commit message: trying to get a proper ur10 model in openrave

File: fh_desc/model.urdf (robot description, URDF)
Before this commit: robot smart_grasping_sandbox, 36 links, 35 joints
Links:
- removed link H1_WR_wrist_base
- removed link world
- added link H1_WR_wrist_base_link, mass 0.126266795472122; collision mesh filename=package://fh_desc/meshes/wrist_base.dae; visual mesh filename=package://fh_desc/meshes/wrist_base.dae
Joints:
- removed joint world_joint
- joint H1_WRJ1: parent H1_WR_wrist_base -> H1_WR_wrist_base_link
- joint H1_WR_wrist_base: child H1_WR_wrist_base -> H1_WR_wrist_base_link
- joint elbow_joint: limit lower=-3.14159265359 upper=3.14159265359 effort=150.0 velocity=3.15 -> lower=-6.28318530718 upper=6.28318530718 effort=150.0 velocity=3.15
- joint shoulder_lift_joint: limit lower=-3.14159265359 upper=3.14159265359 effort=330.0 velocity=2.16 -> lower=-6.28318530718 upper=6.28318530718 effort=330.0 velocity=2.16
- joint shoulder_pan_joint: limit lower=-3.14159265359 upper=3.14159265359 effort=330.0 velocity=2.16 -> lower=-6.28318530718 upper=6.28318530718 effort=330.0 velocity=2.16
- joint wrist_1_joint: limit lower=-3.14159265359 upper=3.14159265359 effort=54.0 velocity=3.2 -> lower=-6.28318530718 upper=6.28318530718 effort=54.0 velocity=3.2
- joint wrist_2_joint: limit lower=-3.14159265359 upper=3.14159265359 effort=54.0 velocity=3.2 -> lower=-6.28318530718 upper=6.28318530718 effort=54.0 velocity=3.2
- joint wrist_3_joint: limit lower=-3.14159265359 upper=3.14159265359 effort=54.0 velocity=3.2 -> lower=-6.28318530718 upper=6.28318530718 effort=54.0 velocity=3.2

Commit message: Migrating to the Hand V2, first import

File: fh_desc/model.urdf (robot description, URDF)
Before this commit: robot smart_grasping_sandbox, 36 links, 35 joints
Links:
- removed link H1_WR_face_plate
- removed link H1_WR_force_torque_sensor
- removed link H1_WR_wrist
- removed link H1_WR_wrist_base
- added link H1_F1_palm_link, mass 0.0341482312344481; visual mesh filename=package://fh_desc/meshes/v2/finger_palm_link.stl
- added link H1_F2_palm_link, mass 0.0341482312344481; visual mesh filename=package://fh_desc/meshes/v2/finger_palm_link.stl
- added link H1_F3_palm_link, mass 0.0341482312344481; visual mesh filename=package://fh_desc/meshes/v2/finger_palm_link.stl
- link H1_F1_base_link: mass 0.206184327436554 -> 0.174652229503358; geometry collision mesh filename=package://fh_desc/meshes/v2/finger_base_link_simple.stl; visual mesh filename=package://fh_desc/meshes/v2/finger_base_link.stl
- link H1_F1_link_1: mass 0.148439137620102 -> 0.0827759744227546; geometry collision mesh filename=package://fh_desc/meshes/v2/finger_prox_link_simple.stl; visual mesh filename=package://fh_desc/meshes/v2/finger_prox_link.stl
- link H1_F1_link_2: mass 0.0468986964963515 -> 0.0270049614151599; geometry collision mesh filename=package://fh_desc/meshes/v2/finger_dist_link_simple.stl; visual mesh filename=package://fh_desc/meshes/v2/finger_dist_link.stl
- link H1_F1_tip: geometry collision mesh filename=package://fh_desc/meshes/omd-d18-tip.stl; visual mesh filename=package://fh_desc/meshes/omd-d18-tip.stl
- link H1_F2_base_link: mass 0.206184327436554 -> 0.174652229503358; geometry collision mesh filename=package://fh_desc/meshes/v2/finger_base_link_simple.stl; visual mesh filename=package://fh_desc/meshes/v2/finger_base_link.stl
- link H1_F2_link_1: mass 0.148439137620102 -> 0.0827759744227546; geometry collision mesh filename=package://fh_desc/meshes/v2/finger_prox_link_simple.stl; visual mesh filename=package://fh_desc/meshes/v2/finger_prox_link.stl
- link H1_F2_link_2: mass 0.0468986964963515 -> 0.0270049614151599; geometry collision mesh filename=package://fh_desc/meshes/v2/finger_dist_link_simple.stl; visual mesh filename=package://fh_desc/meshes/v2/finger_dist_link.stl
- link H1_F2_tip: geometry collision mesh filename=package://fh_desc/meshes/omd-d18-tip.stl; visual mesh filename=package://fh_desc/meshes/omd-d18-tip.stl
- link H1_F3_base_link: mass 0.206184327436554 -> 0.174652229503358; geometry collision mesh filename=package://fh_desc/meshes/v2/finger_base_link_simple.stl; visual mesh filename=package://fh_desc/meshes/v2/finger_base_link.stl
- link H1_F3_link_1: mass 0.148439137620102 -> 0.0827759744227546; geometry collision mesh filename=package://fh_desc/meshes/v2/finger_prox_link_simple.stl; visual mesh filename=package://fh_desc/meshes/v2/finger_prox_link.stl
- link H1_F3_link_2: mass 0.0468986964963515 -> 0.0270049614151599; geometry collision mesh filename=package://fh_desc/meshes/v2/finger_dist_link_simple.stl; visual mesh filename=package://fh_desc/meshes/v2/finger_dist_link.stl
- link H1_F3_tip: geometry collision mesh filename=package://fh_desc/meshes/omd-d18-tip.stl; visual mesh filename=package://fh_desc/meshes/omd-d18-tip.stl
- link H1_base_link: mass 0.802291302622713 -> 0.07527; geometry collision mesh filename=package://fh_desc/meshes/v2/palm_link_simple.stl; visual mesh filename=package://fh_desc/meshes/v2/palm_link.stl
Joints:
- removed joint H1_F1Base
- removed joint H1_F2Base
- removed joint H1_F3Base
- removed joint H1_WRJ1
- removed joint H1_WR_wrist_base
- removed joint H1_WR_wrist_to_ft_sensor
- removed joint H1_WRft_sensor_to_faceplate
- added joint H1_F1J3: type revolute, parent H1_F1_link_1, child H1_F1_link_2, origin xyz=0 0 0.06 rpy=-0.0068649 1.7347E-18 1.6176E-16, axis 1 0 0, limit lower=-1.0471975512 upper=1.57079632679 effort=2 velocity=1.0
- added joint H1_F1Palm: type fixed, parent H1_insert_F1, child H1_F1_palm_link, origin xyz=0 0 0 rpy=0 0 0
- added joint H1_F2J3: type revolute, parent H1_F2_link_1, child H1_F2_link_2, origin xyz=0 0 0.06 rpy=-0.0068649 1.7347E-18 1.6176E-16, axis 1 0 0, limit lower=-1.0471975512 upper=1.57079632679 effort=2 velocity=1.0
- added joint H1_F2Palm: type fixed, parent H1_insert_F2, child H1_F2_palm_link, origin xyz=0 0 0 rpy=0 0 0
- added joint H1_F3J3: type revolute, parent H1_F3_link_1, child H1_F3_link_2, origin xyz=0 0 0.06 rpy=-0.0068649 1.7347E-18 1.6176E-16, axis 1 0 0, limit lower=-1.0471975512 upper=1.57079632679 effort=2 velocity=1.0
- added joint H1_F3Palm: type fixed, parent H1_insert_F3, child H1_F3_palm_link, origin xyz=0 0 0 rpy=0 0 0
- joint H1Base: parent H1_WR_face_plate -> H1_base_attach
- joint H1_F1J1: axis 1 0 0 -> 0 0 1; child H1_F1_link_1 -> H1_F1_base_link; limit lower=-1.57079632679 upper=1.0472 effort=50 velocity=1.0 -> lower=-0.785398163397 upper=0.785398163397 effort=2 velocity=1.0; origin xyz=0 0 0.096 rpy=0 0 0 -> xyz=0 0 0.00016528 rpy=-8.8818E-16 -1.0061E-16 0.022402; parent H1_F1_base_link -> H1_F1_palm_link
- joint H1_F1J2: child H1_F1_link_2 -> H1_F1_link_1; limit lower=-1.04716 upper=1.57075 effort=50 velocity=1.0 -> lower=-1.3962634016 upper=1.0471975512 effort=2 velocity=1.0; origin xyz=0 0 0.06 rpy=0 0 0 -> xyz=0 0.035 0.11683 rpy=0.070695 6.9389E-16 2.0947E-16; parent H1_F1_link_1 -> H1_F1_base_link
- joint H1_F2J1: axis 1 0 0 -> 0 0 1; child H1_F2_link_1 -> H1_F2_base_link; limit lower=-1.57079632679 upper=1.0472 effort=30 velocity=1.0 -> lower=-0.785398163397 upper=0.785398163397 effort=2 velocity=1.0; origin xyz=0 0 0.096 rpy=0 0 0 -> xyz=0 0 0.00016528 rpy=-8.8818E-16 -1.0061E-16 0.022402; parent H1_F2_base_link -> H1_F2_palm_link
- joint H1_F2J2: child H1_F2_link_2 -> H1_F2_link_1; limit lower=-1.04716 upper=1.57075 effort=30 velocity=1.0 -> lower=-1.3962634016 upper=1.0471975512 effort=2 velocity=1.0; origin xyz=0 0 0.06 rpy=0 0 0 -> xyz=0 0.035 0.11683 rpy=0.070695 6.9389E-16 2.0947E-16; parent H1_F2_link_1 -> H1_F2_base_link
- joint H1_F3J1: axis 1 0 0 -> 0 0 1; child H1_F3_link_1 -> H1_F3_base_link; limit lower=-1.57079632679 upper=1.0472 effort=30 velocity=1.0 -> lower=-0.785398163397 upper=0.785398163397 effort=2 velocity=1.0; origin xyz=0 0 0.096 rpy=0 0 0 -> xyz=0 0 0.00016528 rpy=-8.8818E-16 -1.0061E-16 0.022402; parent H1_F3_base_link -> H1_F3_palm_link
- joint H1_F3J2: child H1_F3_link_2 -> H1_F3_link_1; limit lower=-1.04716 upper=1.57075 effort=30 velocity=1.0 -> lower=-1.3962634016 upper=1.0471975512 effort=2 velocity=1.0; origin xyz=0 0 0.06 rpy=0 0 0 -> xyz=0 0.035 0.11683 rpy=0.070695 6.9389E-16 2.0947E-16; parent H1_F3_link_1 -> H1_F3_base_link
- joint H1_dummy_joint_1: axis (none) -> 0 -1 0; origin xyz=0 0.045 0.002 rpy=0 0 0 -> xyz=-0.045 -0.025981 0 rpy=0 0 2.3562
- joint H1_dummy_joint_2: axis (none) -> 0 -1 0; origin xyz=0.038971 -0.0225 0.002 rpy=0 0 3.14159265359 -> xyz=0 0.029019 0 rpy=0 0 0
- joint H1_dummy_joint_3: axis (none) -> 0 -1 0; origin xyz=-0.038971 -0.0225 0.002 rpy=0 0 3.14159265359 -> xyz=0.045 -0.025981 0 rpy=0 0 -2.3562

Commit message: Using simplified meshes for visualisation too

File: fh_desc/model.urdf (robot description, URDF)
Before this commit: robot smart_grasping_sandbox, 35 links, 34 joints
Links:
- link H1_F1_base_link: geometry collision mesh filename=package://fh_desc/meshes/v2/finger_base_link_simple.dae; visual mesh filename=package://fh_desc/meshes/v2/finger_base_link_simple.dae
- link H1_F1_link_1: geometry collision mesh filename=package://fh_desc/meshes/v2/finger_prox_link_simple.dae; visual mesh filename=package://fh_desc/meshes/v2/finger_prox_link_simple.dae
- link H1_F1_link_2: geometry collision mesh filename=package://fh_desc/meshes/v2/finger_dist_link_simple.dae; visual mesh filename=package://fh_desc/meshes/v2/finger_dist_link_simple.dae
- link H1_F1_palm_link: geometry visual mesh filename=package://fh_desc/meshes/v2/finger_palm_link.dae
- link H1_F1_tip: geometry collision mesh filename=package://fh_desc/meshes/omd-d18-tip.dae; visual mesh filename=package://fh_desc/meshes/omd-d18-tip.dae
- link H1_F2_base_link: geometry collision mesh filename=package://fh_desc/meshes/v2/finger_base_link_simple.dae; visual mesh filename=package://fh_desc/meshes/v2/finger_base_link_simple.dae
- link H1_F2_link_1: geometry collision mesh filename=package://fh_desc/meshes/v2/finger_prox_link_simple.dae; visual mesh filename=package://fh_desc/meshes/v2/finger_prox_link.dae
- link H1_F2_link_2: geometry collision mesh filename=package://fh_desc/meshes/v2/finger_dist_link_simple.dae; visual mesh filename=package://fh_desc/meshes/v2/finger_dist_link_simple.dae
- link H1_F2_palm_link: geometry visual mesh filename=package://fh_desc/meshes/v2/finger_palm_link.dae
- link H1_F2_tip: geometry collision mesh filename=package://fh_desc/meshes/omd-d18-tip.dae; visual mesh filename=package://fh_desc/meshes/omd-d18-tip.dae
- link H1_F3_base_link: geometry collision mesh filename=package://fh_desc/meshes/v2/finger_base_link_simple.dae; visual mesh filename=package://fh_desc/meshes/v2/finger_base_link.dae
- link H1_F3_link_1: geometry collision mesh filename=package://fh_desc/meshes/v2/finger_prox_link_simple.dae; visual mesh filename=package://fh_desc/meshes/v2/finger_prox_link_simple.dae
- link H1_F3_link_2: geometry collision mesh filename=package://fh_desc/meshes/v2/finger_dist_link_simple.dae; visual mesh filename=package://fh_desc/meshes/v2/finger_dist_link.dae
- link H1_F3_palm_link: geometry visual mesh filename=package://fh_desc/meshes/v2/finger_palm_link.dae
- link H1_F3_tip: geometry collision mesh filename=package://fh_desc/meshes/omd-d18-tip.dae; visual mesh filename=package://fh_desc/meshes/omd-d18-tip.dae
- link H1_base_link: geometry collision mesh filename=package://fh_desc/meshes/v2/palm_link_simple.dae; visual mesh filename=package://fh_desc/meshes/v2/palm_link_simple.dae
- link base_link: geometry collision mesh filename=package://ur_description/meshes/ur10/collision/base.dae; visual mesh filename=package://ur_description/meshes/ur10/visual/base.dae
- link forearm_link: geometry collision mesh filename=package://ur_description/meshes/ur10/collision/forearm.dae; visual mesh filename=package://ur_description/meshes/ur10/visual/forearm.dae
- link shoulder_link: geometry collision mesh filename=package://ur_description/meshes/ur10/collision/shoulder.dae; visual mesh filename=package://ur_description/meshes/ur10/visual/shoulder.dae
- link upper_arm_link: geometry collision mesh filename=package://ur_description/meshes/ur10/collision/upperarm.dae; visual mesh filename=package://ur_description/meshes/ur10/visual/upperarm.dae
- link wrist_1_link: geometry collision mesh filename=package://ur_description/meshes/ur10/collision/wrist1.dae; visual mesh filename=package://ur_description/meshes/ur10/visual/wrist1.dae
- link wrist_2_link: geometry collision mesh filename=package://ur_description/meshes/ur10/collision/wrist2.dae; visual mesh filename=package://ur_description/meshes/ur10/visual/wrist2.dae
- link wrist_3_link: geometry collision mesh filename=package://ur_description/meshes/ur10/collision/wrist3.dae; visual mesh filename=package://ur_description/meshes/ur10/visual/wrist3.dae

Commit message: fixing dae

File: fh_desc/model.urdf (robot description, URDF)
Before this commit: robot smart_grasping_sandbox, 35 links, 34 joints
Links:
- link H1_F3_link_2: geometry collision mesh filename=package://fh_desc/meshes/v2/finger_dist_link_simple.dae; visual mesh filename=package://fh_desc/meshes/v2/finger_dist_link_simple.dae

Commit message: fixing links to meshes

File: fh_desc/model.urdf (robot description, URDF)
Before this commit: robot smart_grasping_sandbox, 35 links, 34 joints
Links:
- link H1_F2_link_1: geometry collision mesh filename=package://fh_desc/meshes/v2/finger_prox_link_simple.dae; visual mesh filename=package://fh_desc/meshes/v2/finger_prox_link_simple.dae
- link H1_F3_base_link: geometry collision mesh filename=package://fh_desc/meshes/v2/finger_base_link_simple.dae; visual mesh filename=package://fh_desc/meshes/v2/finger_base_link_simple.dae

Commit message: better values for physics

File: fh_desc/model.urdf (robot description, URDF)
Before this commit: robot smart_grasping_sandbox, 35 links, 34 joints
Joints:
- joint H1_F1J1: limit lower=-0.785398163397 upper=0.785398163397 effort=2 velocity=1.0 -> lower=-0.785398163397 upper=0.785398163397 effort=50 velocity=1.0
- joint H1_F1J2: limit lower=-1.3962634016 upper=1.0471975512 effort=2 velocity=1.0 -> lower=-1.3962634016 upper=1.0471975512 effort=50 velocity=1.0
- joint H1_F1J3: limit lower=-1.0471975512 upper=1.57079632679 effort=2 velocity=1.0 -> lower=-1.0471975512 upper=1.57079632679 effort=50 velocity=1.0
- joint H1_F2J1: limit lower=-0.785398163397 upper=0.785398163397 effort=2 velocity=1.0 -> lower=-0.785398163397 upper=0.785398163397 effort=50 velocity=1.0
- joint H1_F2J2: limit lower=-1.3962634016 upper=1.0471975512 effort=2 velocity=1.0 -> lower=-1.3962634016 upper=1.0471975512 effort=50 velocity=1.0
- joint H1_F2J3: limit lower=-1.0471975512 upper=1.57079632679 effort=2 velocity=1.0 -> lower=-1.0471975512 upper=1.57079632679 effort=50 velocity=1.0
- joint H1_F3J1: limit lower=-0.785398163397 upper=0.785398163397 effort=2 velocity=1.0 -> lower=-0.785398163397 upper=0.785398163397 effort=50 velocity=1.0
- joint H1_F3J2: limit lower=-1.3962634016 upper=1.0471975512 effort=2 velocity=1.0 -> lower=-1.3962634016 upper=1.0471975512 effort=50 velocity=1.0
- joint H1_F3J3: limit lower=-1.0471975512 upper=1.57079632679 effort=2 velocity=1.0 -> lower=-1.0471975512 upper=1.57079632679 effort=50 velocity=1.0

Commit message: ball is grasped with the new hand

File: fh_desc/model.urdf (robot description, URDF)
Before this commit: robot smart_grasping_sandbox, 35 links, 34 joints
Joints:
- joint H1_F1J1: limit lower=-0.785398163397 upper=0.785398163397 effort=50 velocity=1.0 -> lower=-0.785398163397 upper=0.785398163397 effort=300 velocity=1.0
- joint H1_F1J2: limit lower=-1.3962634016 upper=1.0471975512 effort=50 velocity=1.0 -> lower=-1.3962634016 upper=1.0471975512 effort=300 velocity=1.0
- joint H1_F1J3: limit lower=-1.0471975512 upper=1.57079632679 effort=50 velocity=1.0 -> lower=-1.0471975512 upper=1.57079632679 effort=300 velocity=1.0
- joint H1_F2J1: limit lower=-0.785398163397 upper=0.785398163397 effort=50 velocity=1.0 -> lower=-0.785398163397 upper=0.785398163397 effort=300 velocity=1.0
- joint H1_F2J2: limit lower=-1.3962634016 upper=1.0471975512 effort=50 velocity=1.0 -> lower=-1.3962634016 upper=1.0471975512 effort=300 velocity=1.0
- joint H1_F2J3: limit lower=-1.0471975512 upper=1.57079632679 effort=50 velocity=1.0 -> lower=-1.0471975512 upper=1.57079632679 effort=300 velocity=1.0
- joint H1_F3J1: limit lower=-0.785398163397 upper=0.785398163397 effort=50 velocity=1.0 -> lower=-0.785398163397 upper=0.785398163397 effort=300 velocity=1.0
- joint H1_F3J2: limit lower=-1.3962634016 upper=1.0471975512 effort=50 velocity=1.0 -> lower=-1.3962634016 upper=1.0471975512 effort=300 velocity=1.0
- joint H1_F3J3: limit lower=-1.0471975512 upper=1.57079632679 effort=50 velocity=1.0 -> lower=-1.0471975512 upper=1.57079632679 effort=300 velocity=1.0
