Commit message: better physics for grasping

File: fh_desc/hand/xacro/0x02000101/0x02000101.xacro (robot description, xacro)
@@ -61,5 +61,5 @@
       <axis xyz="1 0 0" />
       <limit lower="-${pi/2}" upper="1.0472" effort="2" velocity="1.0" />
-      <dynamics damping="0.1"/>
+      <dynamics  damping="0.005" friction="0.005"/>
     </joint>
     <joint name="${hand_id}_${part_id}J2" type="revolute">
@@ -68,6 +68,6 @@
       <parent link="${hand_id}_${part_id}_link_1"/>
       <child link="${hand_id}_${part_id}_link_2"/>
-      <limit lower="-1.04716" upper="1.57075" effort="2" velocity="1.0" />
-      <dynamics damping="0.01"/>
+      <limit lower="-1.04716" upper="1.57075" effort="5." velocity="1.0" />
+      <dynamics  damping="0.005" friction="0.005"/>
     </joint>
     <xacro:if value="${transmission}">

File: fh_desc/hand/xacro/0x02000103/0x02000103.xacro (robot description, xacro)
@@ -39,5 +39,5 @@
       <axis xyz="-1 0 0" />
       <limit lower="-0.785" upper="0.785" effort="20" velocity="0.1" />
-      <dynamic damping="0.1"/>
+      <dynamic  damping="0.005" friction="0.005"/>
     </joint>
     <link name="${hand_id}_${part_id}_force_torque_sensor">

File: fh_desc/hand/xacro/0x1234/0x1234.xacro (robot description, xacro)
@@ -30,6 +30,6 @@
       <insert_block name="origin"/>
       <axis xyz="0 1 0" />
-      <limit lower="0.0" upper="${pi/2}" effort="2" velocity="1.0" />
-      <dynamics damping="0.1"/>
+      <limit lower="0.0" upper="${pi/2}" effort="5." velocity="1.0" />
+      <dynamics  damping="0.005" friction="0.005"/>
     </joint>
   </xacro:macro>

File: fh_desc/hand/xacro/0x1235/0x1235.xacro (robot description, xacro)
@@ -27,6 +27,6 @@
       <insert_block name="origin"/>
       <axis xyz="0 1 0" />
-      <limit lower="0.0" upper="${pi/2}" effort="2" velocity="1.0" />
-      <dynamics damping="0.1"/>
+      <limit lower="0.0" upper="${pi/2}" effort="5." velocity="1.0" />
+      <dynamics  damping="0.005" friction="0.005"/>
     </joint>
   </xacro:macro>
